Commit message: add some seabeds

File: urdf/turbine.xacro (robot description, xacro)
@@ -28,10 +28,10 @@
     <collision>
       <geometry>
-        <mesh filename="file://$(find floatgen)/meshes/base_air.stl"/>
+        <mesh filename="file://$(find floatgen)/meshes/base_air.dae"/>
       </geometry>
     </collision>
     <collision>
       <geometry>
-        <mesh filename="file://$(find floatgen)/meshes/base_water.stl"/>
+        <mesh filename="file://$(find floatgen)/meshes/base_water.dae"/>
       </geometry>
     </collision>

Commit message: separate gz and spawn with arguments

File: urdf/turbine.xacro (robot description, xacro)
@@ -18,20 +18,20 @@
     <visual>
       <geometry>
-        <mesh filename="file://$(find floatgen)/meshes/base_air.dae"/>
+        <mesh filename="package://floatgen/meshes/base_air.dae"/>
       </geometry>
     </visual>
     <visual>
       <geometry>
-        <mesh filename="file://$(find floatgen)/meshes/base_water.dae"/>
+        <mesh filename="package://floatgen/meshes/base_water.dae"/>
       </geometry>
     </visual>
     <collision>
       <geometry>
-        <mesh filename="file://$(find floatgen)/meshes/base_air.dae"/>
+        <mesh filename="package://floatgen/meshes/base_air.dae"/>
       </geometry>
     </collision>
     <collision>
       <geometry>
-        <mesh filename="file://$(find floatgen)/meshes/base_water.dae"/>
+        <mesh filename="package://floatgen/meshes/base_water.dae"/>
       </geometry>
     </collision>
@@ -67,5 +67,5 @@
     <visual>
       <geometry>
-        <mesh filename="file://$(find floatgen)/meshes/pole.dae"  scale="1 1 1"/>
+        <mesh filename="package://floatgen/meshes/pole.dae"  scale="1 1 1"/>
       </geometry>
     </visual>
@@ -81,5 +81,5 @@
     <visual>
       <geometry>
-        <mesh filename="file://$(find floatgen)/meshes/blades.dae"  scale="1 1 1"/>
+        <mesh filename="package://floatgen/meshes/blades.dae"  scale="1 1 1"/>
       </geometry>
     </visual>
